File: PCB/Hackpad.kicad_pcb (KiCad board)
At the start: 2 copper layers, 83.3 x 66.7 mm, 7 parts, among them SW1 SW_Push, SW2 SW_Push, SW3 SW_Push, SW4 SW_Push, U1 XIAO-RP2040-DIP

Commit message: wiring better
Routing:
- net Net-(U1-GPIO2/SCK): track 100.2 -> 24.2 mm
- net Net-(U1-GPIO1/RX): track 156.2 -> 91.8 mm
- net Net-(U1-GPIO3/MOSI): track 109.4 -> 75.4 mm
- net Net-(U1-GPIO4/MISO): track 79.7 -> 52.8 mm
- net +5V: track 72.6 -> 82.5 mm
- net Net-(D2-DIN): track 44.5 -> 40.7 mm

Commit message: lotta stuff
Parts:
- added C1: C, Capacitor_THT:DX_5R5HxxxxU_D11.5mm_P10.00mm, F.Cu at (150.7, 55.9)
- added C2: C_Small, Capacitor_THT:DX_5R5VxxxxU_D11.5mm_P5.00mm, F.Cu at (221.7, 55.0)
Routing:
- net +5V: track 82.5 -> 116.5 mm
- net Net-(U1-GPIO1/RX): track 91.8 -> 82.8 mm
Other:
- board text added: "6-26-2025"

Commit message: attempted changes
Connections:
- C1 pad 2: GND2 -> Net-(D2-VDD)
- C2 pad 1: +5V -> Net-(D1-VDD)
- C2 pad 2: GND3 -> +5V
- D1 pad 4: +5V -> Net-(D1-VDD)
- D2 pad 4: +5V -> Net-(D2-VDD)
Routing:
- net Net-(D1-VDD): track 0.00 -> 84.7 mm
- net Net-(D2-VDD): track 0.00 -> 59.9 mm
- net +5V: track 116.5 -> 92.3 mm, vias 0 -> 1
Changed lines of the file:
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@@
 	(net 16 "unconnected-(U1-GPIO7{slash}SCL-Pad6)")
 	(net 17 "unconnected-(U1-GPIO28{slash}ADC2{slash}A2-Pad3)")
-	(net 18 "GND2")
-	(net 19 "GND3")
+	(net 18 "Net-(D2-VDD)")
+	(net 19 "Net-(D1-VDD)")
 	(footprint "LED_SMD:LED_SK6812MINI_PLCC4_3.5x3.5mm_P1.75mm"
 		(layer "F.Cu")
@@
 			(size 1.6 0.85)
 			(layers "F.Cu" "F.Mask" "F.Paste")
-			(net 4 "+5V")
+			(net 18 "Net-(D2-VDD)")
 			(pinfunction "VDD")
 			(pintype "power_in")
@@
 			(layers "*.Cu" "*.Mask")
 			(remove_unused_layers no)
-			(net 18 "GND2")
+			(net 18 "Net-(D2-VDD)")
 			(pintype "passive")
 		)
@@
 			(size 1.6 0.85)
 			(layers "F.Cu" "F.Mask" "F.Paste")
-			(net 4 "+5V")
+			(net 19 "Net-(D1-VDD)")
 			(pinfunction "VDD")
 			(pintype "power_in")
@@
 			(layers "*.Cu" "*.Mask")
 			(remove_unused_layers no)
-			(net 4 "+5V")
+			(net 19 "Net-(D1-VDD)")
 			(pintype "passive")
 		)
@@
 			(layers "*.Cu" "*.Mask")
 			(remove_unused_layers no)
-			(net 19 "GND3")
+			(net 4 "+5V")
 			(pintype "passive")
 		)
@@
 	)
 	(segment
-		(start 211.93125 72.06875)
-		(end 211.93125 47.83125)
+		(start 184.2605 56.24575)
+		(end 193.3575 47.14875)
 		(width 0.2)
 		(layer "F.Cu")
@@
 	)
 	(segment
-		(start 184.2605 56.24575)
-		(end 193.3575 47.14875)
+		(start 176.026874 56.24575)
+		(end 184.2605 56.24575)
 		(width 0.2)
 		(layer "F.Cu")
@@
 	)
 	(segment
-		(start 176.026874 56.24575)
-		(end 184.2605 56.24575)
+		(start 164.386312 67.886312)
+		(end 176.026874 56.24575)
 		(width 0.2)
 		(layer "F.Cu")
@@
 	(segment
 		(start 164.30625 67.966374)
-		(end 176.026874 56.24575)
+		(end 164.386312 67.886312)
 		(width 0.2)
 		(layer "F.Cu")
@@
 		(net 4)
 	)
+	(via
+		(at 164.386312 67.886312)
+		(size 0.6)
+		(drill 0.3)
+		(layers "F.Cu" "B.Cu")
+		(net 4)
+	)
 	(segment
 		(start 152.25 55.85)
@@
 		(net 9)
 	)
+	(segment
+		(start 211.95 71.85794)
+		(end 211.95 72.1)
+		(width 0.2)
+		(layer "B.Cu")
+		(net 18)
+	)
+	(segment
+		(start 162.79425 53.70575)
+		(end 193.79781 53.70575)
+		(width 0.2)
+		(layer "B.Cu")
+		(net 18)
+	)
+	(segment
+		(start 193.79781 53.70575)
+		(end 211.95 71.85794)
+		(width 0.2)
+		(layer "B.Cu")
+		(net 18)
+	)
+	(segment
+		(start 160.65 55.85)
+		(end 162.79425 53.70575)
+		(width 0.2)
+		(layer "B.Cu")
+		(net 18)
+	)
+	(segment
+		(start 165.25 51.25)
+		(end 163.469728 51.25)
+		(width 0.2)
+		(layer "B.Cu")
+		(net 19)
+	)
+	(segment
+		(start 165.33425 51.16575)
+		(end 165.25 51.25)
+		(width 0.2)
+		(layer "B.Cu")
+		(net 19)
+	)
+	(segment
+		(start 221.65 54.95)
+		(end 217.86575 51.16575)
+		(width 0.2)
+		(layer "B.Cu")
+		(net 19)
+	)
+	(segment
+		(start 163.469728 51.25)
+		(end 159.674 55.045728)
+		(width 0.2)
+		(layer "B.Cu")
+		(net 19)
+	)
+	(segment
+		(start 159.674 55.045728)
+		(end 159.674 62.324057)
+		(width 0.2)
+		(layer "B.Cu")
+		(net 19)
+	)
+	(segment
+		(start 159.674 62.324057)
+		(end 164.987312 67.637369)
+		(width 0.2)
+		(layer "B.Cu")
+		(net 19)
+	)
+	(segment
+		(start 164.987312 71.412688)
+		(end 164.3 72.1)
+		(width 0.2)
+		(layer "B.Cu")
+		(net 19)
+	)
+	(segment
+		(start 217.86575 51.16575)
+		(end 165.33425 51.16575)
+		(width 0.2)
+		(layer "B.Cu")
+		(net 19)
+	)
+	(segment
+		(start 164.987312 67.637369)
+		(end 164.987312 71.412688)
+		(width 0.2)
+		(layer "B.Cu")
+		(net 19)
+	)
 	(embedded_fonts no)

Commit message: fixed a lottta errors-ty meddy
Parts:
- C1: footprint Capacitor_THT:DX_5R5HxxxxU_D11.5mm_P10.00mm -> Capacitor_THT:C_Axial_L3.8mm_D2.6mm_P7.50mm_Horizontal
- C2: footprint Capacitor_THT:DX_5R5VxxxxU_D11.5mm_P5.00mm -> Capacitor_THT:C_Axial_L3.8mm_D2.6mm_P7.50mm_Horizontal
- U1: moved to B.Cu
- moved C2 31.6 mm to (208.2, 83.5), turned to 180 degrees
- moved C1 30.3 mm to (163.6, 83.2)
- moved U1 26.0 mm to (185.9, 80.8), turned to 180 degrees
- moved SW3 19.2 mm to (188.5, 75.7)
- moved SW1 19.1 mm to (188.5, 94.9)
- moved D2 15.3 mm to (204.6, 87.2), turned to 180 degrees
- moved D1 15.1 mm to (167.4, 87.2)
- moved SW4 0.37 mm to (207.7, 94.9)
Connections:
- C1 pad 1: +5V -> GND
- C1 pad 2: Net-(D2-VDD) -> +5V
- C2 pad 1: Net-(D1-VDD) -> GND
- D1 pad 4: Net-(D1-VDD) -> +5V
- D2 pad 4: Net-(D2-VDD) -> +5V
Routing:
- net Net-(D1-VDD): track 84.7 -> 0.00 mm
- net Net-(U1-GPIO3/MOSI): track 75.4 -> 4.86 mm
- net Net-(D2-VDD): track 59.9 -> 0.00 mm
- net Net-(U1-GPIO1/RX): track 82.8 -> 26.8 mm
- net +5V: track 92.3 -> 53.7 mm, vias 1 -> 0
- net Net-(U1-GPIO4/MISO): track 52.8 -> 21.3 mm
- net Net-(D2-DIN): track 40.7 -> 10.6 mm
- net GND: track 102.8 -> 87.6 mm, vias 0 -> 2
- net Net-(U1-GPIO2/SCK): track 24.2 -> 14.1 mm
- net Net-(D1-DIN): track 44.8 -> 40.0 mm, vias 0 -> 2
Other:
- board size 83.3 x 66.7 mm -> 61.5 x 43.8 mm
- board text removed: "6-26-2025"
- board text removed: "Hackpad by Agniva/Knivier"
- board text removed: "XIAO HERE"
