File: PCB/Hackpad.kicad_sch (KiCad schematic)
At the start: 7 parts, among them SW1 SW_Push, SW2 SW_Push, SW3 SW_Push, SW4 SW_Push, U1 XIAO-RP2040-DIP

Commit message: lotta stuff
Parts:
- added C1: C, Capacitor_THT:DX_5R5HxxxxU_D11.5mm_P10.00mm, symbol Device:C
- added C2: C_Small, Capacitor_THT:DX_5R5VxxxxU_D11.5mm_P5.00mm, symbol Device:C_Small
Connections:
- net +5V: now also C1.1, C2.1
- new net GND2: C1.2
- new net GND3: C2.2

Commit message: attempted changes
Connections:
- net GND3 is gone; now on net +5V: C2.2
- net +5V: no longer C2.1, D1.4 (VDD), D2.4 (VDD)
- net GND2: no longer names the net of C1.2
- net GND2: now also D2.4 (VDD)
- new net: C2.1, D1.4 (VDD)
Other:
- moved on the sheet: C1, C2
Changed lines of the file:
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@@
 	(paper "A4")
-	(junction
-		(at 114.3 50.8)
-		(diameter 0)
-		(color 0 0 0 0)
-	)
 	(junction
 		(at 139.7 50.8)
@@
 	)
 	(junction
-		(at 139.7 55.88)
-		(diameter 0)
-		(color 0 0 0 0)
-	)
-	(junction
 		(at 139.7 74.93)
 		(diameter 0)
@@
 	(wire
 		(pts
-			(xy 139.7 55.88) (xy 139.7 59.69)
+			(xy 139.7 50.8) (xy 139.7 53.34)
 		)
 		(stroke
@@
 	(wire
 		(pts
+			(xy 139.7 58.42) (xy 139.7 59.69)
+		)
+		(stroke
+			(width 0)
+			(type default)
+		)
+	)
+	(wire
+		(pts
 			(xy 101.6 67.31) (xy 101.6 114.3)
 		)
@@
 	(wire
 		(pts
-			(xy 139.7 50.8) (xy 139.7 55.88)
-		)
-		(stroke
-			(width 0)
-			(type default)
-		)
-	)
-	(wire
-		(pts
 			(xy 152.4 114.3) (xy 146.05 114.3)
 		)
@@
 	(wire
 		(pts
-			(xy 114.3 50.8) (xy 139.7 50.8)
-		)
-		(stroke
-			(width 0)
-			(type default)
-		)
-	)
-	(wire
-		(pts
 			(xy 146.05 132.08) (xy 146.05 121.92)
 		)
@@
 	(wire
 		(pts
-			(xy 109.22 50.8) (xy 114.3 50.8)
+			(xy 109.22 50.8) (xy 111.76 50.8)
+		)
+		(stroke
+			(width 0)
+			(type default)
+		)
+	)
+	(wire
+		(pts
+			(xy 119.38 50.8) (xy 139.7 50.8)
 		)
 		(stroke
@@
 	)
 	(symbol
-		(lib_id "power:GND3")
-		(at 144.78 55.88 90)
-		(unit 1)
-		(exclude_from_sim no)
-		(in_bom yes)
-		(on_board yes)
-		(dnp no)
-		(fields_autoplaced yes)
-		(property "Reference" "#PWR07"
-			(at 151.13 55.88 0)
-			(effects
-				(font
-					(size 1.27 1.27)
-				)
-				(hide yes)
-			)
-		)
-		(property "Value" "GND3"
-			(at 148.59 55.8799 90)
-			(effects
-				(font
-					(size 1.27 1.27)
-				)
-				(justify right)
-			)
-		)
-		(property "Footprint" ""
-			(at 144.78 55.88 0)
-			(effects
-				(font
-					(size 1.27 1.27)
-				)
-				(hide yes)
-			)
-		)
-		(property "Datasheet" ""
-			(at 144.78 55.88 0)
-			(effects
-				(font
-					(size 1.27 1.27)
-				)
-				(hide yes)
-			)
-		)
-		(property "Description" "Power symbol creates a global label with name \"GND3\" , ground"
-			(at 144.78 55.88 0)
-			(effects
-				(font
-					(size 1.27 1.27)
-				)
-				(hide yes)
-			)
-		)
-		(pin "1"
-		)
-		(instances
-			(project ""
-				(path "/cf02a346-a8bc-4000-87af-25e97e7e97c6"
-					(reference "#PWR07")
-					(unit 1)
-				)
-			)
-		)
-	)
-	(symbol
 		(lib_id "LED:SK6812MINI")
 		(at 109.22 67.31 0)
@@
 	)
 	(symbol
-		(lib_id "power:GND2")
-		(at 114.3 43.18 180)
-		(unit 1)
-		(exclude_from_sim no)
-		(in_bom yes)
-		(on_board yes)
-		(dnp no)
-		(fields_autoplaced yes)
-		(property "Reference" "#PWR06"
-			(at 114.3 36.83 0)
-			(effects
-				(font
-					(size 1.27 1.27)
-				)
-				(hide yes)
-			)
-		)
-		(property "Value" "GND2"
-			(at 114.3 38.1 0)
-			(effects
-				(font
-					(size 1.27 1.27)
-				)
-			)
-		)
-		(property "Footprint" ""
-			(at 114.3 43.18 0)
-			(effects
-				(font
-					(size 1.27 1.27)
-				)
-				(hide yes)
-			)
-		)
-		(property "Datasheet" ""
-			(at 114.3 43.18 0)
-			(effects
-				(font
-					(size 1.27 1.27)
-				)
-				(hide yes)
-			)
-		)
-		(property "Description" "Power symbol creates a global label with name \"GND2\" , ground"
-			(at 114.3 43.18 0)
-			(effects
-				(font
-					(size 1.27 1.27)
-				)
-				(hide yes)
-			)
-		)
-		(pin "1"
-		)
-		(instances
-			(project ""
-				(path "/cf02a346-a8bc-4000-87af-25e97e7e97c6"
-					(reference "#PWR06")
-					(unit 1)
-				)
-			)
-		)
-	)
-	(symbol
 		(lib_id "LED:SK6812MINI")
 		(at 139.7 67.31 0)
@@
 	(symbol
 		(lib_id "Device:C_Small")
-		(at 142.24 55.88 90)
+		(at 139.7 55.88 180)
 		(unit 1)
 		(exclude_from_sim no)
@@
 		(fields_autoplaced yes)
 		(property "Reference" "C2"
-			(at 142.2463 49.53 90)
-			(effects
-				(font
-					(size 1.27 1.27)
-				)
+			(at 142.24 54.6035 0)
+			(effects
+				(font
+					(size 1.27 1.27)
+				)
+				(justify right)
 			)
 		)
 		(property "Value" "C_Small"
-			(at 142.2463 52.07 90)
-			(effects
-				(font
-					(size 1.27 1.27)
-				)
+			(at 142.24 57.1435 0)
+			(effects
+				(font
+					(size 1.27 1.27)
+				)
+				(justify right)
 			)
 		)
 		(property "Footprint" "Capacitor_THT:DX_5R5VxxxxU_D11.5mm_P5.00mm"
-			(at 142.24 55.88 0)
+			(at 139.7 55.88 0)
 			(effects
 				(font
@@
 		)
 		(property "Datasheet" "~"
-			(at 142.24 55.88 0)
+			(at 139.7 55.88 0)
 			(effects
 				(font
@@
 		)
 		(property "Description" "Unpolarized capacitor, small symbol"
-			(at 142.24 55.88 0)
+			(at 139.7 55.88 0)
 			(effects
 				(font
@@
 	(symbol
 		(lib_id "Device:C")
-		(at 114.3 46.99 180)
+		(at 115.57 50.8 270)
 		(unit 1)
 		(exclude_from_sim no)
@@
 		(fields_autoplaced yes)
 		(property "Reference" "C1"
-			(at 118.11 45.7199 0)
-			(effects
-				(font
-					(size 1.27 1.27)
-				)
-				(justify right)
+			(at 115.57 43.18 90)
+			(effects
+				(font
+					(size 1.27 1.27)
+				)
 			)
 		)
 		(property "Value" "C"
-			(at 118.11 48.2599 0)
-			(effects
-				(font
-					(size 1.27 1.27)
-				)
-				(justify right)
+			(at 115.57 45.72 90)
+			(effects
+				(font
+					(size 1.27 1.27)
+				)
 			)
 		)
 		(property "Footprint" "Capacitor_THT:DX_5R5HxxxxU_D11.5mm_P10.00mm"
-			(at 113.3348 43.18 0)
+			(at 111.76 51.7652 0)
 			(effects
 				(font
@@
 		)
 		(property "Datasheet" "~"
-			(at 114.3 46.99 0)
+			(at 115.57 50.8 0)
 			(effects
 				(font
@@
 		)
 		(property "Description" "Unpolarized capacitor"
-			(at 114.3 46.99 0)
-			(effects
-				(font
+			(at 115.57 50.8 0)
+			(effects
+				(font

Commit message: fixed a lottta errors-ty meddy
Parts:
- C1: footprint Capacitor_THT:DX_5R5HxxxxU_D11.5mm_P10.00mm -> Capacitor_THT:C_Axial_L3.8mm_D2.6mm_P7.50mm_Horizontal
- C2: footprint Capacitor_THT:DX_5R5VxxxxU_D11.5mm_P5.00mm -> Capacitor_THT:C_Axial_L3.8mm_D2.6mm_P7.50mm_Horizontal
Connections:
- net +5V: now also C1.2, D1.4 (VDD), D2.4 (VDD); no longer C1.1
- net GND: now also C1.1, C2.1
Other:
- moved on the sheet: C1, C2
Changed lines of the file:
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@@
+	)
+	(junction
+		(at 139.7 55.88)
+		(diameter 0)
+		(color 0 0 0 0)
+	)
+	(junction
+		(at 115.57 50.8)
+		(diameter 0)
+		(color 0 0 0 0)
 	)
 	(junction
@@
 	(wire
 		(pts
-			(xy 139.7 50.8) (xy 139.7 53.34)
-		)
-		(stroke
-			(width 0)
-			(type default)
-		)
-	)
-	(wire
-		(pts
 			(xy 69.85 130.81) (xy 69.85 137.16)
 		)
@@
 	(wire
 		(pts
-			(xy 139.7 58.42) (xy 139.7 59.69)
+			(xy 139.7 50.8) (xy 139.7 55.88)
 		)
 		(stroke
@@
 	(wire
 		(pts
+			(xy 139.7 55.88) (xy 139.7 59.69)
+		)
+		(stroke
+			(width 0)
+			(type default)
+		)
+	)
+	(wire
+		(pts
+			(xy 115.57 50.8) (xy 139.7 50.8)
+		)
+		(stroke
+			(width 0)
+			(type default)
+		)
+	)
+	(wire
+		(pts
 			(xy 96.52 86.36) (xy 96.52 132.08)
 		)
@@
 	(wire
 		(pts
-			(xy 109.22 50.8) (xy 111.76 50.8)
-		)
-		(stroke
-			(width 0)
-			(type default)
-		)
-	)
-	(wire
-		(pts
-			(xy 119.38 50.8) (xy 139.7 50.8)
+			(xy 109.22 50.8) (xy 115.57 50.8)
 		)
 		(stroke
@@
 	(symbol
 		(lib_id "power:GND")
+		(at 115.57 43.18 180)
+		(unit 1)
+		(exclude_from_sim no)
+		(in_bom yes)
+		(on_board yes)
+		(dnp no)
+		(fields_autoplaced yes)
+		(property "Reference" "#PWR07"
+			(at 115.57 36.83 0)
+			(effects
+				(font
+					(size 1.27 1.27)
+				)
+				(hide yes)
+			)
+		)
+		(property "Value" "GND"
+			(at 115.57 38.1 0)
+			(effects
+				(font
+					(size 1.27 1.27)
+				)
+			)
+		)
+		(property "Footprint" ""
+			(at 115.57 43.18 0)
+			(effects
+				(font
+					(size 1.27 1.27)
+				)
+				(hide yes)
+			)
+		)
+		(property "Datasheet" ""
+			(at 115.57 43.18 0)
+			(effects
+				(font
+					(size 1.27 1.27)
+				)
+				(hide yes)
+			)
+		)
+		(property "Description" "Power symbol creates a global label with name \"GND\" , ground"
+			(at 115.57 43.18 0)
+			(effects
+				(font
+					(size 1.27 1.27)
+				)
+				(hide yes)
+			)
+		)
+		(pin "1"
+		)
+		(instances
+			(project "Hackpad"
+				(path "/cf02a346-a8bc-4000-87af-25e97e7e97c6"
+					(reference "#PWR07")
+					(unit 1)
+				)
+			)
+		)
+	)
+	(symbol
+		(lib_id "power:GND")
 		(at 139.7 74.93 0)
 		(unit 1)
@@
 	)
 	(symbol
+		(lib_id "power:GND")
+		(at 144.78 55.88 90)
+		(unit 1)
+		(exclude_from_sim no)
+		(in_bom yes)
+		(on_board yes)
+		(dnp no)
+		(fields_autoplaced yes)
+		(property "Reference" "#PWR06"
+			(at 151.13 55.88 0)
+			(effects
+				(font
+					(size 1.27 1.27)
+				)
+				(hide yes)
+			)
+		)
+		(property "Value" "GND"
+			(at 148.59 55.8799 90)
+			(effects
+				(font
+					(size 1.27 1.27)
+				)
+				(justify right)
+			)
+		)
+		(property "Footprint" ""
+			(at 144.78 55.88 0)
+			(effects
+				(font
+					(size 1.27 1.27)
+				)
+				(hide yes)
+			)
+		)
+		(property "Datasheet" ""
+			(at 144.78 55.88 0)
+			(effects
+				(font
+					(size 1.27 1.27)
+				)
+				(hide yes)
+			)
+		)
+		(property "Description" "Power symbol creates a global label with name \"GND\" , ground"
+			(at 144.78 55.88 0)
+			(effects
+				(font
+					(size 1.27 1.27)
+				)
+				(hide yes)
+			)
+		)
+		(pin "1"
+		)
+		(instances
+			(project ""
+				(path "/cf02a346-a8bc-4000-87af-25e97e7e97c6"
+					(reference "#PWR06")
+					(unit 1)
+				)
+			)
+		)
+	)
+	(symbol
 		(lib_id "LED:SK6812MINI")
 		(at 109.22 67.31 0)
@@
 	(symbol
 		(lib_id "Device:C_Small")
-		(at 139.7 55.88 180)
+		(at 142.24 55.88 270)
 		(unit 1)
 		(exclude_from_sim no)
@@
 		(fields_autoplaced yes)
 		(property "Reference" "C2"
-			(at 142.24 54.6035 0)
-			(effects
-				(font
-					(size 1.27 1.27)
-				)
-				(justify right)
+			(at 142.2336 49.53 90)
+			(effects
+				(font
+					(size 1.27 1.27)
+				)
 			)
 		)
 		(property "Value" "C_Small"
-			(at 142.24 57.1435 0)
-			(effects
-				(font
-					(size 1.27 1.27)
-				)
-				(justify right)
-			)
-		)
-		(property "Footprint" "Capacitor_THT:DX_5R5VxxxxU_D11.5mm_P5.00mm"
-			(at 139.7 55.88 0)
+			(at 142.2336 52.07 90)
+			(effects
+				(font
+					(size 1.27 1.27)
+				)
+			)
+		)
+		(property "Footprint" "Capacitor_THT:C_Axial_L3.8mm_D2.6mm_P7.50mm_Horizontal"
+			(at 142.24 55.88 0)
 			(effects
 				(font
@@
 		)
 		(property "Datasheet" "~"
-			(at 139.7 55.88 0)
+			(at 142.24 55.88 0)
 			(effects
 				(font
@@
 		)
 		(property "Description" "Unpolarized capacitor, small symbol"
-			(at 139.7 55.88 0)
+			(at 142.24 55.88 0)
 			(effects
 				(font
@@
 		)
 		(instances
-			(project ""
+			(project "Hackpad"
 				(path "/cf02a346-a8bc-4000-87af-25e97e7e97c6"
 					(reference "C2")
@@
 	(symbol
 		(lib_id "Device:C")
-		(at 115.57 50.8 270)
+		(at 115.57 46.99 0)
 		(unit 1)
 		(exclude_from_sim no)
@@
 		(fields_autoplaced yes)
 		(property "Reference" "C1"
-			(at 115.57 43.18 90)
-			(effects
-				(font
-					(size 1.27 1.27)
-				)
+			(at 119.38 45.7199 0)
+			(effects
+				(font
+					(size 1.27 1.27)
+				)
+				(justify left)
 			)
 		)
 		(property "Value" "C"
-			(at 115.57 45.72 90)
-			(effects
-				(font
-					(size 1.27 1.27)
-				)
-			)
-		)
-		(property "Footprint" "Capacitor_THT:DX_5R5HxxxxU_D11.5mm_P10.00mm"
-			(at 111.76 51.7652 0)
+			(at 119.38 48.2599 0)
+			(effects
+				(font
+					(size 1.27 1.27)
+				)
+				(justify left)
+			)
+		)
+		(property "Footprint" "Capacitor_THT:C_Axial_L3.8mm_D2.6mm_P7.50mm_Horizontal"
+			(at 116.5352 50.8 0)
 			(effects
 				(font
@@
 		)
 		(property "Datasheet" "~"
-			(at 115.57 50.8 0)
+			(at 115.57 46.99 0)
 			(effects
 				(font
@@
 		)
 		(property "Description" "Unpolarized capacitor"
-			(at 115.57 50.8 0)
+			(at 115.57 46.99 0)
 			(effects
 				(font
@@
 		)
 		(instances
-			(project ""
+			(project "Hackpad"
 				(path "/cf02a346-a8bc-4000-87af-25e97e7e97c6"
 					(reference "C1")
